File: P5/P5.kicad_pcb (KiCad board)
At the start: 2 copper layers, 500 x 310 mm, 127 parts, among them J1 1-10, J2 Conn_01x10, J3 Conn_01x10, J4 Conn_01x10, J5 Conn_01x05, Q1 BC1, SW1 SW_Rotary1x3, SW10 SW_SPDT, SW11 SW_SPDT, SW12 SW_SPST, SW2 SW_SPDT, SW3 SW_SPDT, SW4 SW_Rotary1x3, SW5 SW_Rotary1x3, SW6 SW_Rotary1x3, SW7 SW_SPDT, SW8 SW_SPDT, SW8B1 SW_SPDT, SW9 SW_SPST, U1 TL072, U2 TL072, U3 LM741, U4 TL072, U5 4070, U6 4006, U7 LM741

Commit message: Upgrade P5 to Kicad9
Parts:
- J1: value 1-10 -> Conn_01x10
