File: P5/P5.kicad_pcb (KiCad board)
At the start: 2 copper layers, 500 x 310 mm, 127 parts, among them J1 Conn_01x10, J2 Conn_01x10, J3 Conn_01x10, J4 Conn_01x10, J5 Conn_01x05, Q1 BC1, SW1 SW_Rotary1x3, SW10 SW_SPDT, SW11 SW_SPDT, SW12 SW_SPST, SW2 SW_SPDT, SW3 SW_SPDT, SW4 SW_Rotary1x3, SW5 SW_Rotary1x3, SW6 SW_Rotary1x3, SW7 SW_SPDT, SW8 SW_SPDT, SW8B1 SW_SPDT, SW9 SW_SPST, U1 TL072, U2 TL072, U3 LM741, U4 TL072, U5 4070, U6 4006, U7 LM741

Commit message: Update P5 layout
Parts:
- C15: footprint Capacitor_THT:CP_Radial_D5.0mm_P2.50mm -> Capacitor_THT:CP_Radial_D8.0mm_P5.00mm
- J1: value Conn_01x10 -> 1-10
- moved R48 28.3 mm to (79.3, 163.3)
- moved R47 28.2 mm to (69.1, 168.5)
- moved R41 26.1 mm to (67.5, 106.0)
- moved R42 26.1 mm to (77.7, 100.9)
- moved R44 14.6 mm to (77.7, 121.2)
- moved R45 14.6 mm to (67.5, 126.3)
- moved R50 13.0 mm to (79.3, 183.7)
- moved R51 12.9 mm to (69.1, 188.8)
- moved R25 9.84 mm to (343.8, 266.0), turned to -90 degrees
- moved R49 8.35 mm to (79.3, 173.5)
- moved R52 8.35 mm to (69.1, 178.6)
- moved R43 5.97 mm to (77.7, 111.1)
- moved R46 5.97 mm to (67.5, 116.1)
- moved SW9 4.14 mm to (323.0, 276.1)
- moved SW11 1.62 mm to (420.8, 276.0)
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Connections:
- J2 pad 2: /12_VCA_D -> /14_VCA_R
- J2 pad 4: /14_VCA_R -> /12_VCA_D
Routing:
- net GND: track 793.0 -> 1975.0 mm, vias 0 -> 3
- net -15V: track 503.8 -> 916.1 mm, vias 0 -> 1
- net /18_NOISE_VOLUME: track 0.00 -> 356.2 mm
- net /10_PITCH_TRACK_VCF: track 0.00 -> 341.5 mm
- net /19_DEPTH: track 0.00 -> 294.8 mm
- net /9_PITCH_TRACK_VCF_ADSR: track 0.00 -> 260.6 mm
- net /8_VCF_R: track 0.00 -> 245.0 mm, vias 0 -> 1
- net /14_VCA_R: track 0.00 -> 244.1 mm, vias 0 -> 1
- net /7_VCF_S: track 0.00 -> 182.6 mm, vias 0 -> 1
- net /13_VCA_S: track 0.00 -> 181.1 mm, vias 0 -> 1
- net +15V: track 347.2 -> 512.4 mm
- net /20_RESONANCE_CONTROL: track 0.00 -> 162.9 mm
- net /6_VCF_D: track 0.00 -> 137.7 mm, vias 0 -> 1
- net /12_VCA_D: track 0.00 -> 136.7 mm, vias 0 -> 1
- net Net-(ZD1-K): track 0.00 -> 123.1 mm, vias 0 -> 1
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