File: P5/P5.kicad_pcb (KiCad board)
At the start: 2 copper layers, 500 x 310 mm, 127 parts, among them J1 1-10, J2 Conn_01x10, J3 Conn_01x10, J4 Conn_01x10, J5 Conn_01x05, Q1 BC1, SW1 SW_Rotary1x3, SW10 SW_SPDT, SW11 SW_SPDT, SW12 SW_SPST, SW2 SW_SPDT, SW3 SW_SPDT, SW4 SW_Rotary1x3, SW5 SW_Rotary1x3, SW6 SW_Rotary1x3, SW7 SW_SPDT, SW8 SW_SPDT, SW8B1 SW_SPDT, SW9 SW_SPST, U1 TL072, U2 TL072, U3 LM741, U4 TL072, U5 4070, U6 4006, U7 LM741

Commit message: Update P5 layout
Parts:
- C10, C11, C12, C9: footprint Capacitor_THT:CP_Radial_D5.0mm_P2.50mm -> Capacitor_THT:CP_Radial_D8.0mm_P5.00mm
- C7: footprint Capacitor_THT:C_Rect_L7.0mm_W3.5mm_P2.50mm_P5.00mm -> Capacitor_THT:CP_Radial_D10.0mm_P5.00mm
- moved SW8B1 50.3 mm to (343.8, 223.6), turned to 180 degrees
- moved R38 21.7 mm to (333.9, 208.8), turned to 90 degrees
- moved D1 21.0 mm to (63.6, 84.4), turned to 0 degrees
- moved R48 20.4 mm to (79.3, 183.7)
- moved R50 20.4 mm to (79.3, 163.3)
- moved R47 20.3 mm to (69.1, 188.8)
- moved R51 20.3 mm to (69.1, 168.5)
- moved R41 20.3 mm to (67.5, 126.3)
- moved R42 20.3 mm to (77.7, 121.2)
- moved R44 20.3 mm to (77.7, 100.9)
- moved R45 20.3 mm to (67.5, 106.0)
- moved SW3 6.17 mm to (49.1, 233.4), turned to 180 degrees
- moved PR2 5.12 mm to (168.6, 202.3), turned to 0 degrees
- moved D2 3.95 mm to (81.3, 84.5)
- moved C6 3.70 mm to (225.5, 264.4)
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Connections:
- C1 pad 2: Net-(U1B-+) -> Net-(U1B--)
- C3 pad 2: Net-(U4B-+) -> Net-(U4B--)
- R23 pad 1: Net-(U4B-+) -> Net-(U4B--)
- R25 pad 1: Net-(U1C-V+) -> +15V
- R26 pad 1: Net-(U1C-V-) -> -15V
- R4 pad 1: Net-(U1B-+) -> Net-(U1B--)
- SW6 pad 1: Net-(PR2-Pad2) -> Net-(PR3-Pad1)
- SW6 pad 3: Net-(PR3-Pad1) -> Net-(PR2-Pad2)
- U1 pad 4: Net-(U1C-V-) -> -15V
- U1 pad 5: Net-(U1B-+) -> GND
- U1 pad 6: GND -> Net-(U1B--)
- U1 pad 8: Net-(U1C-V+) -> +15V
- U2 pad 4: Net-(U1C-V-) -> -15V
- U2 pad 8: Net-(U1C-V+) -> +15V
- U4 pad 4: Net-(U1C-V-) -> -15V
- U4 pad 5: Net-(U4B-+) -> GND
- U4 pad 6: GND -> Net-(U4B--)
- U4 pad 8: Net-(U1C-V+) -> +15V
- U7 pad 4: +15V -> -15V
- U7 pad 7: -15V -> +15V
Routing:
- net GND: track 1975.0 -> 3231.4 mm, vias 3 -> 21
- net +15V: track 512.4 -> 1664.3 mm, vias 0 -> 6
- net -15V: track 916.1 -> 1698.5 mm, vias 1 -> 13
- net /39_VCO2_SAW: track 0.00 -> 495.1 mm
- net /22_SYNC: track 0.00 -> 495.0 mm
- net Net-(R15-Pad2): track 0.00 -> 480.7 mm
- net /40_VCO2_TRI: track 0.00 -> 475.3 mm
- net /41_VCO2_SQR: track 0.00 -> 447.1 mm
- net /42_VCO1_SAW: track 0.00 -> 390.9 mm
- net /27_VCO2_PWM_MOD: track 0.00 -> 372.5 mm
- net /43_VCO1_TRI: track 0.00 -> 370.8 mm
- net /44_VCO1_SQR: track 0.00 -> 355.5 mm
- net /25_VCO2_VOL: track 0.00 -> 344.5 mm, vias 0 -> 2
- net /21_VIBRATO: track 0.00 -> 342.9 mm
- net /28_VCO1_PWM_MOD: track 0.00 -> 319.8 mm
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Other:
- outline, holes or cut-outs redrawn

Commit message: Finish P5 layout
Parts:
- moved R31 0.21 mm to (172.0, 255.0)
Connections:
- C7 pad 1: VCC -> +15V
- R31 pad 1: VCC -> +15V
- R33 pad 2: VCC -> +15V
- U5 pad 1: VCC -> +15V
- U5 pad 6: VCC -> +15V
Routing:
- net +15V: track 1664.3 -> 2076.2 mm, vias 6 -> 12
- net GND: track 3231.4 -> 3490.0 mm, vias 21 -> 22
- net -15V: track 1698.5 -> 1849.3 mm
- net VCC: track 20.3 -> 0.00 mm
- net Net-(PR1-Pad1): track 0.00 -> 9.57 mm
- net Net-(R44-Pad2): track 13.8 -> 18.8 mm
Other:
- board size 500 x 310 mm -> 436.5 x 270.4 mm
