File: P3/P3.kicad_pcb (KiCad board)
At the start: 2 copper layers, 349.2 x 160 mm, 116 parts, among them J1 Conn_01x10, J2 Conn_01x05, J3 Conn_01x10, J4 Conn_01x05, J5 Conn_02x07_Counter_Clockwise, J6 Screw_Terminal_01x02, U1 SN75107B, U10 74LS08, U11 7425, U12 74LS32, U13 74LS193, U14 74LS153, U15 74LS74, U16 74LS93, U17 74LS244, U18 74LS367, U19 74LS367, U2 74LS175, U20 74LS32, U21 74LS74, U22 74LS266, U23 74LS266, U24 6810-Memory_RAM-eti-polysynth, U25 74LS08, U26 74LS08, U27 CD4051B, U28 74LS259, U29 74LS13, U3 74LS74, U30 74LS93, U31 74LS93, U32 74LS93, U33 74LS42, U34 74LS32, U35 74LS04, U36 7404, U37 4041, U38 4041, U39 TL072, U4 D2102, U40 TL082, U41 TL082, U42 TL082, U43 TL082, U44 L7805, U5 74LS00, U6 74LS04, U7 74LS10, U8 74LS00, U9 74LS32

Commit message: Routing P3/updating footprints to Kicad9
Parts:
- moved C23 3.47 mm to (343.8, 130.5), turned to 180 degrees
- moved C14 3.24 mm to (44.2, 115.5), turned to 180 degrees
- moved C25 2.87 mm to (321.8, 201.8)
- moved C20 2.23 mm to (223.2, 139.2), turned to 180 degrees
- moved C24 2.08 mm to (197.0, 193.5)
- moved U20 1.58 mm to (57.5, 95.2)
- moved U16 1.44 mm to (57.5, 121.2)
- moved U10 1.39 mm to (36.2, 120.9)
- moved U21 1.39 mm to (36.2, 94.5)
- moved U32 1.36 mm to (130.5, 147.2)
- moved C19 1.32 mm to (171.0, 167.2), turned to 180 degrees
- moved U7 1.28 mm to (57.2, 172.8)
- moved U12 1.25 mm to (57.5, 147.2)
- moved U9 1.21 mm to (36.2, 147.2)
- moved U15 1.20 mm to (109.5, 173.0)
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Routing:
- net +5V: track 402.3 -> 1252.6 mm, vias 5 -> 13
- net GND: track 357.8 -> 966.7 mm, vias 1 -> 3
- net /M: track 292.1 -> 475.7 mm, vias 7 -> 8
- net -5V: track 282.5 -> 406.3 mm, vias 3 -> 6
- net GNDA: track 159.4 -> 174.7 mm
- net Net-(U33-A3): track 38.6 -> 29.4 mm
- net Net-(U18-OEb): track 345.0 -> 351.3 mm, vias 5 -> 7
- net Net-(U14-Zb): track 71.5 -> 68.6 mm
- net Net-(U10-Pad5): track 120.9 -> 123.6 mm
- net Net-(U10-Pad10): track 46.8 -> 44.2 mm
- net Net-(U7-Pad6): track 86.9 -> 89.5 mm
- net /IC2_11: track 301.7 -> 304.2 mm
- net Net-(U21A-Q): track 87.2 -> 89.7 mm
- net /K5: track 17.8 -> 20.2 mm
- net /A2: track 381.9 -> 379.5 mm
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- removed copper zone on B.Cu, net +5V
- removed copper zone on F.Cu, net GND

Commit message: Routing P3
Parts:
- removed H3, H5: MountingHole, MountingHole:MountingHole_3.2mm_M3_DIN965_Pad
- J6: footprint TerminalBlock:TerminalBlock_Altech_AK300-2_P5.00mm -> TerminalBlock_Altech:Altech_AK100_1x02_P5.00mm
- moved C27 10.0 mm to (325.8, 213.2), turned to 180 degrees
- moved J6 5.08 mm to (333.0, 82.8)
- moved C13 4.14 mm to (300.8, 98.5)
- moved C12 3.94 mm to (293.0, 98.5)
- moved C15 1.37 mm to (57.2, 169.5)
- moved H1 1.15 mm to (19.0, 71.0)
- moved H4 0.96 mm to (175.5, 145.0)
- moved C25 0.50 mm to (321.8, 202.2)
- moved U38 0.45 mm to (274.0, 186.2)
- moved H2 0.32 mm to (19.8, 214.9)
- moved HS1 0.05 mm to (296.9, 82.8)
Routing:
- net GND: track 966.7 -> 1742.4 mm, vias 3 -> 1
- net GNDA: track 174.7 -> 412.3 mm
- net +3.3VDAC: track 6.45 -> 112.2 mm
- net +5V: track 1252.6 -> 1349.5 mm, vias 13 -> 14
- net Net-(R21-Pad2): track 21.2 -> 34.0 mm, vias 0 -> 1
- net Net-(R23-Pad2): track 21.2 -> 30.0 mm
- net Net-(U18-OEb): track 351.3 -> 357.1 mm
- net Net-(D1-K): track 33.1 -> 27.7 mm
- net Net-(D2-K): track 16.6 -> 11.5 mm
- net Net-(R19-Pad2): track 12.9 -> 16.5 mm
- net /~{F2}: track 221.2 -> 219.3 mm, vias 3 -> 2
- net Net-(U21B-Q): track 147.4 -> 148.9 mm
- net /1_VOICE: track 226.8 -> 227.8 mm
- net /K5: track 20.2 -> 19.4 mm
- net Net-(D3-K): track 140.6 -> 139.8 mm
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
Commit message: Routing P3 done
Parts:
- removed H6: MountingHole, MountingHole:MountingHole_3.2mm_M3_DIN965_Pad
- moved C24 13.8 mm to (210.8, 195.0), turned to -90 degrees
Routing:
- net GND: track 1742.4 -> 1879.8 mm
- net GNDA: track 412.3 -> 457.4 mm, vias 0 -> 3
- net /IC2-D2: track 67.3 -> 59.4 mm
- net /D2: track 217.0 -> 218.7 mm
- net Net-(U18-O5b): track 440.2 -> 441.7 mm
- net -5V: track 405.6 -> 406.3 mm
- added copper zone on B.Cu, net GNDA
