File: P3/P3.kicad_sch (KiCad schematic)
At the start: 116 parts, among them J1 Conn_01x10, J2 Conn_01x05, J3 Conn_01x10, J4 Conn_01x05, J5 Conn_02x07_Counter_Clockwise, J6 Screw_Terminal_01x02, U1 SN75107B, U10 74LS08, U11 7425, U12 74LS32, U13 74LS193, U14 74LS153, U15 74LS74, U16 74LS93, U17 74LS244, U18 74LS367, U19 74LS367, U2 74LS175, U20 74LS32, U21 74LS74, U22 74LS266, U23 74LS266, U24 6810-Memory_RAM-eti-polysynth, U25 74LS08, U26 74LS08, U27 CD4051B, U28 74LS259, U29 74LS13, U3 74LS74, U30 74LS93, U31 74LS93, U32 74LS93, U33 74LS42, U34 74LS32, U35 74LS04, U36 7404, U37 4041, U38 4041, U39 TL072, U4 D2102, U40 TL082, U41 TL082, U42 TL082, U43 TL082, U44 L7805, U5 74LS00, U6 74LS04, U7 74LS10, U8 74LS00, U9 74LS32

Commit message: Routing P3
Parts:
- removed H3, H5: MountingHole, MountingHole:MountingHole_3.2mm_M3_DIN965_Pad, symbol Mechanical:MountingHole
- H1, H2, H4, H6, H7, H8: now left out of the parts list
- J6: footprint TerminalBlock:TerminalBlock_Altech_AK300-2_P5.00mm -> TerminalBlock_Altech:Altech_AK100_1x02_P5.00mm
- U24: footprint Package_DIP:DIP-24_W10.16mm_LongPads -> Package_DIP:DIP-24_W15.24mm_LongPads
Other:
- moved on the sheet: C12, C9

Commit message: Routing P3 done
Parts:
- removed H6: MountingHole, MountingHole:MountingHole_3.2mm_M3_DIN965_Pad, symbol Mechanical:MountingHole
Changed lines of the file:
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@@
-	(symbol
-		(lib_id "Mechanical:MountingHole")
-		(at 494.03 360.68 0)
-		(unit 1)
-		(exclude_from_sim no)
-		(in_bom no)
-		(on_board yes)
-		(dnp no)
-		(property "Reference" "H6"
-			(at 496.57 359.41 0)
-			(effects
-				(font
-					(size 1.27 1.27)
-				)
-				(justify left)
-			)
-		)
-		(property "Value" "MountingHole"
-			(at 496.57 360.68 0)
-			(effects
-				(font
-					(size 1.27 1.27)
-				)
-				(justify left)
-			)
-		)
-		(property "Footprint" "MountingHole:MountingHole_3.2mm_M3_DIN965_Pad"
-			(at 494.03 360.68 0)
-			(effects
-				(font
-					(size 1.27 1.27)
-				)
-				(hide yes)
-			)
-		)
-		(property "Datasheet" ""
-			(at 494.03 360.68 0)
-			(effects
-				(font
-					(size 1.27 1.27)
-				)
-				(hide yes)
-			)
-		)
-		(property "Description" ""
-			(at 494.03 360.68 0)
-			(effects
-				(font
-					(size 1.27 1.27)
-				)
-			)
-		)
-		(instances
-			(project "P3"
-				(path "/b94c0cc6-780f-4e33-9eb2-931a72fdabfa"
-					(reference "H6")
-					(unit 1)
-				)
-			)
-		)
-	)
 	(symbol
 		(lib_id "Mechanical:MountingHole")
