File: P1-2/P1-2.kicad_sch (KiCad schematic)
At the start: 91 parts, among them J1 Conn_02x07_Odd_Even, J2 Conn_01x11_Pin, J3 Conn_01x11_Pin, Q1 BC212L, SW1 Conn_01x01_Pin, SW10 Conn_01x01_Pin, SW11 Conn_01x01_Pin, SW12 Conn_01x01_Pin, SW13 Conn_01x01_Pin, SW14 Conn_01x01_Pin, SW15 Conn_01x01_Pin, SW16 Conn_01x01_Pin, SW17 Conn_01x01_Pin, SW18 Conn_01x01_Pin, SW19 Conn_01x01_Pin, SW2 Conn_01x01_Pin, SW20 Conn_01x01_Pin, SW21 Conn_01x01_Pin, SW22 Conn_01x01_Pin, SW23 Conn_01x01_Pin, SW24 Conn_01x01_Pin, SW25 Conn_01x01_Pin, SW26 Conn_01x01_Pin, SW27 Conn_01x01_Pin, SW28 Conn_01x01_Pin, SW29 Conn_01x01_Pin, SW3 Conn_01x01_Pin, SW30 Conn_01x01_Pin, SW31 Conn_01x01_Pin, SW32 Conn_01x01_Pin, SW33 Conn_01x01_Pin, SW34 Conn_01x01_Pin, SW35 Conn_01x01_Pin, SW36 Conn_01x01_Pin, SW37 Conn_01x01_Pin, SW38 Conn_01x01_Pin, SW39 Conn_01x01_Pin, SW4 Conn_01x01_Pin, SW40 Conn_01x01_Pin, SW41 Conn_01x01_Pin, SW42 Conn_01x01_Pin, SW43 Conn_01x01_Pin, SW44 Conn_01x01_Pin, SW45 Conn_01x01_Pin, SW46 Conn_01x01_Pin, SW47 Conn_01x01_Pin, SW48 Conn_01x01_Pin, SW49 Conn_01x01_Pin, SW5 Conn_01x01_Pin, SW6 Conn_01x01_Pin, SW7 Conn_01x01_Pin, SW8 Conn_01x01_Pin, SW9 Conn_01x01_Pin, U1 4051, U2 4051, U3 4051, U4 4051, U5 4051, U6 4051, U7 4051, U8 74LS42

Commit message: Update footprints from library on P1-2
Parts:
- H1, H2, H3, H4, H5, H6: now left out of the parts list
