File: P4/P4.kicad_pcb (KiCad board)
At the start: 2 copper layers, 359.7 x 231.5 mm, 128 parts, among them J1 Conn_01x10, J11 Conn_01x10, J12 Conn_01x10, J13 Conn_01x25, J14 Conn_01x25, J15 Conn_01x25, J16 Conn_01x25, J17 Conn_01x25, J18 Conn_01x25, J19 Conn_01x25, J2 Conn_01x10, J20 Conn_01x25, J21 Conn_01x25, J22 Conn_01x25, J26 Conn_01x01, J3 Conn_01x10, J4 Conn_01x10, J5 Conn_01x05, J6 Conn_01x10, J7 Conn_01x10, J8 Conn_01x03, J9 Conn_01x03, Q1 BC212L, Q2 BC212L, Q3 TIP42, Q4 TIP41, U1 LM723_DIP14, U10 LM13600, U11 LF353, U12 LM741, U13 LM13600, U2 LM741, U3 L7905, U4 LM1458, U5 LM1458, U6 LF353, U7 LM13600, U8 LF353, U9 LF353

Commit message: Update P4 layout
Parts:
- added J10: Conn_01x25, Connector_PinSocket_2.54mm:PinSocket_1x25_P2.54mm_Vertical, F.Cu at (390.2, 213.2)
- added J23: Conn_01x10, Connector_PinHeader_2.54mm:PinHeader_1x10_P2.54mm_Vertical, F.Cu at (392.8, 124.8)
- moved R44 29.5 mm to (145.9, 159.0)
- moved J22 13.7 mm to (385.2, 162.9)
- moved J21 12.3 mm to (385.2, 226.4)
- moved U3 0.89 mm to (67.9, 115.8)
- moved HS3 0.76 mm to (70.3, 107.2)
- moved CA19 0.47 mm to (136.0, 212.2)
- moved Q1 0.38 mm to (166.8, 70.0)
- moved R15 0.28 mm to (79.8, 151.0)
- moved R18 0.24 mm to (72.2, 140.8)
Connections:
- J13 pad 2: (no net) -> unconnected-(J13-Pin_2-Pad2)
- J13 pad 5: (no net) -> unconnected-(J13-Pin_5-Pad5)
- J15 pad 2: (no net) -> unconnected-(J15-Pin_2-Pad2)
- J15 pad 5: (no net) -> unconnected-(J15-Pin_5-Pad5)
- J17 pad 2: (no net) -> unconnected-(J17-Pin_2-Pad2)
- J17 pad 5: (no net) -> unconnected-(J17-Pin_5-Pad5)
- J19 pad 2: (no net) -> unconnected-(J19-Pin_2-Pad2)
- J19 pad 5: (no net) -> unconnected-(J19-Pin_5-Pad5)
- J21 pad 12: (no net) -> unconnected-(J21-Pin_12-Pad12)
- J21 pad 2: (no net) -> unconnected-(J21-Pin_2-Pad2)
- J21 pad 3: (no net) -> unconnected-(J21-Pin_3-Pad3)
- J21 pad 4: (no net) -> unconnected-(J21-Pin_4-Pad4)
- J21 pad 5: (no net) -> unconnected-(J21-Pin_5-Pad5)
- J22 pad 12: (no net) -> unconnected-(J22-Pin_12-Pad12)
- J22 pad 17: (no net) -> unconnected-(J22-Pin_17-Pad17)
- J3 pad 3: (no net) -> unconnected-(J3-Pin_3-Pad3)
- J6 pad 6: (no net) -> unconnected-(J6-Pin_6-Pad6)
- R44 pad 2: (no net) -> Earth_Protective
- U1 pad 1: (no net) -> unconnected-(U1-NC-Pad1)
- U1 pad 14: (no net) -> unconnected-(U1-NC-Pad14)
- U1 pad 8: (no net) -> unconnected-(U1-NC-Pad8)
- U1 pad 9: (no net) -> unconnected-(U1-VZ-Pad9)
- U10 pad 10: (no net) -> unconnected-(U10-Pad10)
- U10 pad 15: (no net) -> unconnected-(U10A-DIODE_BIAS-Pad15)
- U10 pad 2: (no net) -> unconnected-(U10C-DIODE_BIAS-Pad2)
- U10 pad 7: (no net) -> unconnected-(U10-Pad7)
- U10 pad 8: (no net) -> unconnected-(U10-Pad8)
- U10 pad 9: (no net) -> unconnected-(U10-Pad9)
- U12 pad 1: (no net) -> unconnected-(U12-NULL-Pad1)
- U12 pad 5: (no net) -> unconnected-(U12-NULL-Pad5)
- U12 pad 8: (no net) -> unconnected-(U12-NC-Pad8)
- U13 pad 10: (no net) -> unconnected-(U13-Pad10)
- U13 pad 12: (no net) -> unconnected-(U13-Pad12)
- U13 pad 13: (no net) -> unconnected-(U13A---Pad13)
- U13 pad 14: (no net) -> unconnected-(U13A-+-Pad14)
- U13 pad 15: (no net) -> unconnected-(U13A-DIODE_BIAS-Pad15)
- U13 pad 16: (no net) -> unconnected-(U13-Pad16)
- U13 pad 7: (no net) -> unconnected-(U13-Pad7)
- U13 pad 8: (no net) -> unconnected-(U13-Pad8)
- U13 pad 9: (no net) -> unconnected-(U13-Pad9)
- U2 pad 1: (no net) -> unconnected-(U2-NULL-Pad1)
- U2 pad 5: (no net) -> unconnected-(U2-NULL-Pad5)
- U2 pad 8: (no net) -> unconnected-(U2-NC-Pad8)
- U7 pad 10: (no net) -> unconnected-(U7-Pad10)
- U7 pad 15: (no net) -> unconnected-(U7A-DIODE_BIAS-Pad15)
- U7 pad 2: (no net) -> unconnected-(U7C-DIODE_BIAS-Pad2)
- U7 pad 7: (no net) -> unconnected-(U7-Pad7)
- U7 pad 8: (no net) -> unconnected-(U7-Pad8)
- U7 pad 9: (no net) -> unconnected-(U7-Pad9)
Routing:
- net /42_G4: track 56.2 -> 661.2 mm, vias 0 -> 2
- net /42_G3: track 28.2 -> 588.0 mm, vias 0 -> 2
- net +15V: track 707.0 -> 1213.2 mm, vias 0 -> 2
- net /42_G2: track 39.8 -> 531.7 mm, vias 0 -> 2
- net /3_L4: track 15.3 -> 256.9 mm
- net /6_L2: track 51.9 -> 293.1 mm
- net /2_L3: track 57.0 -> 298.1 mm
- net /5_L1: track 18.7 -> 258.6 mm
- net /18_NOISE_VOLUME: track 143.0 -> 334.5 mm
- net /1_PITCH_BEND: track 206.6 -> 387.5 mm, vias 1 -> 2
- net /38_ADSR_TRACK_CVF: track 158.5 -> 297.4 mm, vias 1 -> 2
- net /42_G1: track 132.5 -> 257.6 mm
- net GND: track 1701.6 -> 1810.1 mm, vias 6 -> 4
- net /39_ADSR_~{CONT}: track 173.2 -> 263.0 mm, vias 0 -> 1
- net /12_ADSR3_ON_OFF: track 187.6 -> 130.7 mm, vias 2 -> 1
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Other:
- board text added: "+15V"
- board text added: "-15V"
- board text added: "-5V"
- board text added: "A1"
- board text added: "A2"
- board text added: "ADSR_CONT"
- board text added: "ADSR_ON_OFF"
- board text added: "ADSR_TRACK_VCF"
- board text added: "ADSR_~{CONT}"
- board text added: "D1"
- board text added: "D2"
- board text added: "G1"
- board text added: "G2"
- board text added: "G3"
- board text added: "G4"
- board text added: "GND"
- board text added: "KEYBOARD_PITCH"
- board text added: "N/C"
- board text added: "NOISE"
- board text added: "OUTPUT"
- board text added: "PITCH_BEND"
- board text added: "Q"
- board text added: "R1"
- board text added: "R2"
- board text added: "S1"
- board text added: "S2"
- board text added: "SYNC"
- board text added: "TRANSPOSE"
- board text added: "VCA_ADSR_TRACK"
- board text added: "VCF_FREQUENCY"
- board text added: "VCF_PITCH_TRACK"
- board text added: "VCF_SWEEP_ADSR"
- board text added: "VCF_SWEEP_DEPTH"
- board text added: "VCO1_MOD"
- board text added: "VCO1_SAW"
- board text added: "VCO1_SQR"
- board text added: "VCO1_TRI"
- board text added: "VCO1_TUNE"
- board text added: "VCO1_VOL"
- board text added: "VCO2_MOD"
- board text added: "VCO2_SAW"
- board text added: "VCO2_SQR"
- board text added: "VCO2_TRI"
- board text added: "VCO2_TUNE"
- board text added: "VCO2_VOL"
- board text added: "VIBRATO_DEPTH"
