File: P4/P4.kicad_sch (KiCad schematic)
At the start: 128 parts, among them J1 Conn_01x10, J11 Conn_01x10, J12 Conn_01x10, J13 Conn_01x25, J14 Conn_01x25, J15 Conn_01x25, J16 Conn_01x25, J17 Conn_01x25, J18 Conn_01x25, J19 Conn_01x25, J2 Conn_01x10, J20 Conn_01x25, J21 Conn_01x25, J22 Conn_01x25, J26 Conn_01x01, J3 Conn_01x10, J4 Conn_01x10, J5 Conn_01x05, J6 Conn_01x10, J7 Conn_01x10, J8 Conn_01x03, J9 Conn_01x03, Q1 BC212L, Q2 BC212L, Q3 TIP42, Q4 TIP41, U1 LM723_DIP14, U10 LM13600, U11 LF353, U12 LM741, U13 LM13600, U2 LM741, U3 L7905, U4 LM1458, U5 LM1458, U6 LF353, U7 LM13600, U8 LF353, U9 LF353

Commit message: Update P4 layout
Parts:
- added J10: Conn_01x25, Connector_PinSocket_2.54mm:PinSocket_1x25_P2.54mm_Vertical, symbol Connector_Generic:Conn_01x25
- added J23: Conn_01x10, Connector_PinHeader_2.54mm:PinHeader_1x10_P2.54mm_Vertical, symbol Connector_Generic:Conn_01x10
- H1: footprint MountingHole:MountingHole_3.2mm_M3_Pad -> (none); now left out of the parts list
- H10, H2, H3, H4, H5, H6, H7, H8, H9, J26: now left out of the parts list
- J13, J14, J15, J16, J17, J18, J19, J20: footprint Connector_PinSocket_2.54mm:PinSocket_1x25_P2.54mm_Vertical -> Connector_PinSocket_4.00mm:PinSocket_1x25_P4.00mm_Vertical
Connections:
- net 10_PITCH_TRACK_VCF: now also J10.21 (Pin_21)
- net 10_VCO2_TRI: now also J10.6 (Pin_6)
- net 11_VCO2_SAW: now also J10.7 (Pin_7)
- net 12_VCA_R: now also J23.2 (Pin_2)
- net 13_TRANSPOSE: now also J10.8 (Pin_8)
- net 13_VCA_S: now also J23.3 (Pin_3)
- net 14_VCA_D: now also J23.4 (Pin_4)
- net 15_SYNC: now also J10.10 (Pin_10)
- net 16_VCA_A: now also J23.5 (Pin_5)
- net 16_VIBRATO_DEPTH: now also J10.11 (Pin_11)
- net 17_VCO1_MOD: now also J10.12 (Pin_12)
- net 18_NOISE_VOLUME: now also J10.22 (Pin_22)
- net 18_VCO2_MOD: now also J10.13 (Pin_13)
- net 19_DEPTH: now also J10.20 (Pin_20)
- net 19_VCO1_VOL: now also J10.14 (Pin_14)
- net 1_PITCH_BEND: now also J10.3 (Pin_3)
- net 20_RESONANCE_CONTROL: now also J10.19 (Pin_19)
- net 20_VCO2_VOL: now also J10.15 (Pin_15)
- net 27_VCF_SWEEP_ADSR: now also J10.17 (Pin_17)
- net 28_VCF_FREQUENCY: now also J10.18 (Pin_18)
- net 2_ADSR_TRACK_VCA: now also J23.1 (Pin_1)
- net 38_ADSR_TRACK_CVF: now also J10.23 (Pin_23)
- net 39_ADSR_~{CONT}: now also J10.25 (Pin_25)
- net 3_ADRS_CONT_VCA: now also J10.24 (Pin_24)
- net 41_VCO2_SQR: now also J10.5 (Pin_5)
- net 42_VCO1_SAW: now also J10.4 (Pin_4)
- net 43_VCO1_TRI: now also J10.1 (Pin_1)
- net 44_VCO1_SQR: now also J10.2 (Pin_2)
- net 47_VCF_ADSR_A: now also J23.9 (Pin_9)
- net 48_VCF_ADSR_D: now also J23.8 (Pin_8)
- net 49_VCF_ADSR_S: now also J23.7 (Pin_7)
- net 50_VCF_ADSR_R: now also J23.6 (Pin_6)
- net GND: now also J10.16 (Pin_16)
- no-connect marks 43 -> 45

Commit message: Update P4 layout
Parts:
- J23: footprint Connector_PinHeader_2.54mm:PinHeader_1x10_P2.54mm_Vertical -> Connector_PinHeader_2.54mm:PinHeader_1x09_P2.54mm_Vertical; symbol Connector_Generic:Conn_01x10 -> Connector_Generic:Conn_01x09
Connections:
- net 12_VCA_R: now also J23.5 (Pin_5); no longer J23.2 (Pin_2)
- net 13_VCA_S: now also J23.4 (Pin_4); no longer J23.3 (Pin_3)
- net 14_VCA_D: now also J23.3 (Pin_3); no longer J23.4 (Pin_4)
- net 16_VCA_A: now also J23.2 (Pin_2); no longer J23.5 (Pin_5)
- net 39_ADSR_~{CONT}: now also J10.24 (Pin_24); no longer J10.25 (Pin_25)
- net 3_ADRS_CONT_VCA: now also J10.25 (Pin_25); no longer J10.24 (Pin_24)
- no-connect marks 45 -> 44
Changed lines of the file:
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@@
 	)
 	(no_connect
-		(at 524.51 302.26)
-	)
-	(no_connect
 		(at 494.03 294.64)
 	)
@@
 	(polyline
 		(pts
-			(xy 523.24 184.15) (xy 523.24 336.55)
+			(xy 523.24 196.85) (xy 523.24 349.25)
 		)
 		(stroke
@@
 	)
 	(label "41_VCA_ADSR_TRACK"
-		(at 524.51 279.4 0)
+		(at 524.51 292.1 0)
 		(effects
 			(font
@@
 	)
 	(label "47_VCF_ADSR_A"
-		(at 524.51 299.72 0)
+		(at 524.51 312.42 0)
 		(effects
 			(font
@@
 	)
 	(label "48_VCF_ADSR_D"
-		(at 524.51 297.18 0)
+		(at 524.51 309.88 0)
 		(effects
 			(font
@@
 	)
 	(label "40_ADSR_CONT"
-		(at 524.51 274.32 0)
+		(at 524.51 276.86 0)
 		(effects
 			(font
@@
 	)
 	(label "46_VCA_ADSR_R"
-		(at 524.51 281.94 0)
+		(at 524.51 302.26 0)
 		(effects
 			(font
@@
 	)
 	(label "39_ADSR_~{CONT}"
-		(at 524.51 276.86 0)
+		(at 524.51 274.32 0)
 		(effects
 			(font
@@
 	)
 	(label "49_VCF_ADSR_S"
-		(at 524.51 294.64 0)
+		(at 524.51 307.34 0)
 		(effects
 			(font
@@
 	)
 	(label "45_VCA_ADSR_S"
-		(at 524.51 284.48 0)
+		(at 524.51 299.72 0)
 		(effects
 			(font
@@
 	)
 	(label "44_VCA_ADSR_D"
-		(at 524.51 287.02 0)
+		(at 524.51 297.18 0)
 		(effects
 			(font
@@
 	)
 	(label "50_VCF_ADSR_R"
-		(at 524.51 292.1 0)
+		(at 524.51 304.8 0)
 		(effects
 			(font
@@
 	)
 	(label "43_VCA_ADSR_A"
-		(at 524.51 289.56 0)
+		(at 524.51 294.64 0)
 		(effects
 			(font
@@
 	)
 	(symbol
-		(lib_id "Connector_Generic:Conn_01x10")
-		(at 519.43 289.56 0)
+		(lib_id "Connector_Generic:Conn_01x09")
+		(at 519.43 302.26 0)
 		(mirror y)
 		(unit 1)
@@
 		(fields_autoplaced yes)
 		(property "Reference" "J23"
-			(at 516.89 289.5599 0)
+			(at 519.43 285.75 0)
 			(effects
 				(font
 					(size 1.27 1.27)
 				)
-				(justify left)
 			)
 		)
 		(property "Value" "Conn_01x10"
-			(at 516.89 292.0999 0)
+			(at 519.43 288.29 0)
 			(effects
 				(font
 					(size 1.27 1.27)
 				)
-				(justify left)
 			)
 		)
-		(property "Footprint" "Connector_PinHeader_2.54mm:PinHeader_1x10_P2.54mm_Vertical"
-			(at 519.43 289.56 0)
+		(property "Footprint" "Connector_PinHeader_2.54mm:PinHeader_1x09_P2.54mm_Vertical"
+			(at 519.43 302.26 0)
 			(effects
 				(font
@@
 			)
 		)
-		(property "Datasheet" ""
-			(at 519.43 289.56 0)
+		(property "Datasheet" "~"
+			(at 519.43 302.26 0)
 			(effects
 				(font
@@
 			)
 		)
-		(property "Description" ""
-			(at 519.43 289.56 0)
+		(property "Description" "Generic connector, single row, 01x09, script generated (kicad-library-utils/schlib/autogen/connector/)"
+			(at 519.43 302.26 0)
 			(effects
 				(font
 					(size 1.27 1.27)
 				)
+				(hide yes)
 			)
 		)
 		(pin "1"
 		)
-		(pin "10"
-		)
 		(pin "2"

Commit message: Finish P4
Parts:
- C10: footprint Capacitor_THT:CP_Radial_D6.3mm_P2.50mm -> Capacitor_THT:CP_Radial_D8.0mm_P5.00mm
- C11, C7, C9: footprint Capacitor_THT:CP_Radial_D6.3mm_P2.50mm -> Capacitor_THT:CP_Radial_D5.0mm_P2.50mm
- H1: footprint (none) -> MountingHole:MountingHole_3.2mm_M3_Pad
Changed lines of the file:
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@@
 			)
 		)
-		(property "Footprint" "Capacitor_THT:CP_Radial_D6.3mm_P2.50mm"
+		(property "Footprint" "Capacitor_THT:CP_Radial_D5.0mm_P2.50mm"
 			(at 553.72 116.84 0)
 			(effects
@@
 			)
 		)
-		(property "Footprint" "Capacitor_THT:CP_Radial_D6.3mm_P2.50mm"
+		(property "Footprint" "Capacitor_THT:CP_Radial_D8.0mm_P5.00mm"
 			(at 535.94 76.2 0)
 			(effects
@@
 		(exclude_from_sim no)
 		(in_bom yes)
-		(on_board yes)
+		(on_board no)
 		(dnp no)
 		(property "Reference" "R44"
@@
 			)
 		)
-		(property "Footprint" "Capacitor_THT:CP_Radial_D6.3mm_P2.50mm"
+		(property "Footprint" "Capacitor_THT:CP_Radial_D5.0mm_P2.50mm"
 			(at 450.85 60.96 0)
 			(effects
@@
 			)
 		)
-		(property "Footprint" "Capacitor_THT:CP_Radial_D6.3mm_P2.50mm"
+		(property "Footprint" "Capacitor_THT:CP_Radial_D5.0mm_P2.50mm"
 			(at 525.78 53.34 0)
 			(effects
@@
 			)
 		)
-		(property "Footprint" ""
+		(property "Footprint" "MountingHole:MountingHole_3.2mm_M3_Pad"
 			(at 222.25 331.47 0)
 			(effects
@@
 		(on_board yes)
 		(dnp no)
+		(fields_autoplaced yes)
 		(property "Reference" "RV_PITCH_BEND1"
-			(at 35.56 334.01 0)
+			(at 35.56 334.0099 0)
 			(effects
 				(font
@@
 		)
 		(property "Value" "R_POT"
-			(at 35.56 335.28 0)
+			(at 35.56 336.5499 0)
 			(effects
 				(font
