File: voicecard/voicecard.kicad_pcb (KiCad board)
At the start: 2 copper layers, 236.8 x 126.6 mm, 187 parts, among them J2 Conn_01x25_Pin, J3 Conn_01x25_Pin, Q1 BF244C, Q2 BF244C, Q3 BF244C, Q4 BC212, Q5 BC212, Q6 BC212, Q7 BC212, Q8 BC212, Q9 BC212, U1 AS3340, U10 LM13700, U11 NE5532, U12 AS3310, U13 AS3310, U2 4016, U3 4016, U4 AS3340, U5 LM13700, U6 CA3080, U7 LM741, U8 LM13700, U9 NE5532

Commit message: Update voicecard layout
Parts:
- moved J2 36.3 mm to (214.0, 149.0)
- moved J3 36.3 mm to (149.5, 149.0)
- moved R10 13.1 mm to (42.1, 47.8), turned to -90 degrees
- moved R14 12.5 mm to (68.8, 47.5), turned to -90 degrees
- moved R96 12.4 mm to (224.5, 40.8), turned to 180 degrees
- moved C15 3.70 mm to (178.7, 102.9), turned to -45 degrees
- moved CP16 3.69 mm to (190.8, 107.0), turned to 90 degrees
- moved CP29 2.77 mm to (244.2, 105.5)
- moved CP28 2.62 mm to (229.8, 104.0)
- moved CP11 1.99 mm to (148.2, 132.8)
- moved CP14 1.65 mm to (174.2, 105.8)
- moved CP21 1.47 mm to (175.7, 58.8)
- moved CP12 1.46 mm to (157.5, 132.8)
- moved R72 1.37 mm to (169.2, 145.5)
- moved CP22 1.27 mm to (205.0, 47.2)
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Routing:
- net /KEY_PITCH: track 0.00 -> 405.3 mm, vias 0 -> 6
- net /VCF_PITCH_TRACK: track 0.00 -> 307.3 mm, vias 0 -> 2
- net Net-(CP22-Pad1): track 0.00 -> 21.6 mm
- net Net-(R96-Pad2): track 0.00 -> 5.53 mm

Commit message: Update voicecard layout
Parts:
- RV5: value 100k -> 22k
- moved RV6 88.3 mm to (177.0, 43.8)
- moved RV8 71.5 mm to (189.0, 114.2)
- moved RV4 65.4 mm to (242.0, 113.5)
- moved RV7 65.3 mm to (176.8, 114.0)
- moved RV5 41.4 mm to (230.3, 114.2)
- moved R28 35.9 mm to (88.0, 86.5), turned to -90 degrees
- moved R29 34.4 mm to (54.1, 98.5), turned to 0 degrees
- moved R71 14.3 mm to (165.4, 129.5), turned to -90 degrees
- moved R80 13.3 mm to (144.1, 102.7), turned to -90 degrees
- moved R84 13.2 mm to (168.2, 91.8), turned to -90 degrees
- moved R68 13.2 mm to (127.5, 145.5), turned to 90 degrees
- moved R50 13.1 mm to (126.0, 62.8), turned to 180 degrees
- moved R56 13.0 mm to (145.2, 79.3), turned to 180 degrees
- moved R46 13.0 mm to (112.2, 38.5), turned to 180 degrees
- moved R66 12.8 mm to (115.7, 132.7), turned to -90 degrees
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- renumbered R29 to R28, R28 to R29
Connections:
- CP16 pad 1: -5V -> GND
- CP16 pad 2: GND -> -5V
- CP29 pad 1: -5V -> GND
- CP29 pad 2: GND -> -5V
- R10 pad 2: Net-(U11A--) -> Net-(Q2-S)
- R14 pad 2: Net-(U11B--) -> Net-(Q3-S)
- R50 pad 2: Net-(R50-Pad2) -> Net-(U10A--)
- R53 pad 1: Net-(R50-Pad2) -> Net-(U10A--)
- R91 pad 2: -15V -> +15V
- U11 pad 2: Net-(U11A--) -> Net-(Q2-S)
- U11 pad 6: Net-(U11B--) -> Net-(Q3-S)
Routing:
- net GND: track 0.00 -> 618.4 mm, vias 0 -> 10
- net +15V: track 0.00 -> 587.3 mm, vias 0 -> 6
- net -15V: track 0.00 -> 586.0 mm, vias 0 -> 11
- net Net-(R72-Pad2): track 0.00 -> 154.9 mm, vias 0 -> 2
- net -5V: track 0.00 -> 138.0 mm, vias 0 -> 4
- net Net-(R73-Pad1): track 0.00 -> 126.9 mm, vias 0 -> 2
- net /VCO2_INPUT: track 0.00 -> 122.8 mm
- net /VCO1_INPUT: track 0.00 -> 104.8 mm
- net Net-(U5C-+): track 0.00 -> 102.8 mm, vias 0 -> 2
- net Net-(R81-Pad2): track 0.00 -> 92.3 mm
- net Net-(Q5-B): track 0.00 -> 84.1 mm, vias 0 -> 2
- net Net-(U10A--): track 0.00 -> 73.8 mm
- net Net-(U5A-+): track 0.00 -> 69.6 mm
- net /VCO1_PULSE_OUT: track 0.00 -> 65.1 mm
- net /TRANSPOSE: track 0.00 -> 60.7 mm
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