File: voicecard/voicecard.kicad_pcb (KiCad board)
At the start: 2 copper layers, 236.8 x 126.6 mm, 187 parts, among them J2 Conn_01x25_Pin, J3 Conn_01x25_Pin, Q1 BF244C, Q2 BF244C, Q3 BF244C, Q4 BC212, Q5 BC212, Q6 BC212, Q7 BC212, Q8 BC212, Q9 BC212, U1 AS3340, U10 LM13700, U11 NE5532, U12 AS3310, U13 AS3310, U2 4016, U3 4016, U4 AS3340, U5 LM13700, U6 CA3080, U7 LM741, U8 LM13700, U9 NE5532

Commit message: Update voicecard layout
Parts:
- moved R98 12.8 mm to (230.4, 67.8), turned to 180 degrees
- moved R4 12.7 mm to (39.4, 105.0), turned to 180 degrees
- moved R64 5.10 mm to (112.0, 125.5), turned to 0 degrees
- moved Q6 5.08 mm to (116.9, 113.0), turned to 0 degrees
- moved RV5 4.68 mm to (230.8, 109.5)
- moved RV2 4.22 mm to (128.4, 123.0)
- moved RV4 4.00 mm to (242.0, 109.5)
Routing:
- net /IC12_PIN2: track 58.2 -> 211.1 mm
- net Net-(Q6-C): track 4.10 -> 112.6 mm
- net GND: track 618.4 -> 720.8 mm, vias 10 -> 14
- net /GATE: track 9.82 -> 92.0 mm, vias 0 -> 4
- net -15V: track 586.0 -> 666.3 mm, vias 11 -> 13
- net +15V: track 587.3 -> 647.4 mm
- net /IC13_PIN10: track 0.00 -> 59.9 mm
- net Net-(Q2-D): track 24.5 -> 77.0 mm
- net -5V: track 138.0 -> 178.0 mm
- net /VCO1_SAW_OUT: track 0.00 -> 34.8 mm
- net Net-(U10A-+): track 44.6 -> 79.1 mm
- net /IC13_PIN2: track 0.00 -> 27.7 mm
- net /PITCH_BEND: track 0.00 -> 26.9 mm
- net /VCO1_TRIANGLE_OUT: track 0.00 -> 23.6 mm
- net Net-(Q6-B): track 0.00 -> 22.9 mm
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
Commit message: Update voicecard layout
Parts:
- CP14: footprint Capacitor_THT:CP_Radial_D5.0mm_P2.50mm -> Capacitor_THT:CP_Radial_D8.0mm_P3.50mm
- CP21: footprint Capacitor_THT:CP_Radial_D5.0mm_P2.50mm -> Capacitor_THT:CP_Radial_D8.0mm_P5.00mm
- CP22: footprint Capacitor_THT:CP_Radial_D5.0mm_P2.50mm -> Capacitor_THT:CP_Radial_D8.0mm_P3.80mm
- CP28: footprint Capacitor_THT:CP_Radial_D5.0mm_P2.50mm -> Capacitor_THT:CP_Radial_Tantal_D5.5mm_P5.00mm
- RV1, RV2, RV3, RV4, RV5, RV7, RV8: footprint Potentiometer_THT:Potentiometer_Bourns_3266Y_Vertical -> Potentiometer_THT:Potentiometer_Bourns_3299Y_Vertical
- RV6, RV9: footprint Potentiometer_THT:Potentiometer_Bourns_3266Y_Vertical -> Potentiometer_THT:Potentiometer_Bourns_3266P_Horizontal
- moved RV6 8.25 mm to (176.8, 52.0), turned to -90 degrees
- moved C15 5.53 mm to (181.2, 110.2), turned to 90 degrees
- moved R78 5.31 mm to (173.8, 125.8)
- moved Q8 5.13 mm to (232.9, 70.6), turned to 180 degrees
- moved C30 4.67 mm to (238.2, 118.0), turned to 180 degrees
- moved R85 3.15 mm to (184.8, 104.5)
- moved R104 2.48 mm to (211.5, 101.0)
- moved CP16 2.41 mm to (192.0, 104.7)
- moved RV4 2.25 mm to (242.0, 111.8)
- moved RV5 2.25 mm to (230.8, 111.8)
- moved C27 1.95 mm to (216.5, 104.5)
- moved C25 1.90 mm to (216.8, 83.5)
- moved CP21 1.80 mm to (177.0, 60.0)
- moved C24 1.75 mm to (209.8, 83.5)
- moved R101 1.75 mm to (213.2, 81.2)
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Connections:
- U2 pad 7: -15V -> GND
- U3 pad 7: -15V -> GND
Routing:
- net GND: track 720.8 -> 965.2 mm, vias 14 -> 18
- net /VCA_ADSR_TRACK: track 0.00 -> 113.8 mm
- net +15V: track 647.4 -> 724.5 mm, vias 6 -> 8
- net /VCO1_PWM: track 15.4 -> 75.8 mm
- net -5V: track 178.0 -> 234.8 mm
- net Net-(R86-Pad2): track 0.00 -> 55.3 mm
- net /GATE: track 92.0 -> 146.6 mm
- net /ADSR_ON/OFF: track 8.34 -> 49.4 mm
- net /ADSR_CONT: track 0.00 -> 39.3 mm
- net Net-(R94-Pad2): track 0.00 -> 39.2 mm, vias 0 -> 2
- net /VCO2_PWM: track 17.6 -> 51.3 mm
- net /HF_TRACK_VCO1: track 0.00 -> 31.1 mm
- net Net-(R95-Pad2): track 0.00 -> 27.1 mm
- net Net-(Q5-B): track 85.6 -> 112.2 mm
- net /VCO2_SAW_OUT: track 0.00 -> 25.9 mm, vias 0 -> 1
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