File: voicecard/voicecard.kicad_pcb (KiCad board)
At the start: 2 copper layers, 236.8 x 126.6 mm, 187 parts, among them J2 Conn_01x25_Pin, J3 Conn_01x25_Pin, Q1 BF244C, Q2 BF244C, Q3 BF244C, Q4 BC212, Q5 BC212, Q6 BC212, Q7 BC212, Q8 BC212, Q9 BC212, U1 AS3340, U10 LM13700, U11 NE5532, U12 AS3310, U13 AS3310, U2 4016, U3 4016, U4 AS3340, U5 LM13700, U6 CA3080, U7 LM741, U8 LM13700, U9 NE5532

Commit message: Finish voicecard layout
Parts:
- moved J3 14.2 mm to (135.3, 149.0)
- moved R65 7.79 mm to (119.2, 135.9), turned to 180 degrees
- moved R67 5.60 mm to (125.1, 145.4)
- moved R76 5.02 mm to (187.2, 145.2)
- moved R43 4.02 mm to (104.3, 123.8)
- moved R40 3.85 mm to (91.6, 135.9)
- moved R41 3.75 mm to (91.6, 132.0)
- moved R42 3.72 mm to (104.3, 128.1)
- moved R66 3.52 mm to (119.2, 132.0), turned to 180 degrees
- moved R77 3.39 mm to (197.0, 142.0)
- moved R68 2.70 mm to (130.2, 145.5)
- moved R114 2.34 mm to (200.8, 140.0)
- moved R113 2.22 mm to (200.8, 136.2)
- moved R49 1.25 mm to (126.0, 59.0)
- moved R70 1.15 mm to (160.6, 145.3)
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Routing:
- net GND: track 965.2 -> 1212.3 mm
- net -15V: track 642.1 -> 821.2 mm, vias 11 -> 10
- net /VCO1_SQR: track 0.00 -> 146.6 mm
- net /VCO1_TRI: track 0.00 -> 143.8 mm
- net /ADSR_TRACK_VCF: track 0.00 -> 126.0 mm
- net /ADSR_ON/OFF: track 49.4 -> 173.2 mm
- net /VCO2_SQR: track 0.00 -> 121.1 mm
- net /SYNC: track 0.00 -> 117.4 mm, vias 0 -> 4
- net /VCO1_SAW: track 0.00 -> 113.3 mm
- net /VCO2_TRI: track 0.00 -> 112.3 mm
- net /VCO2_SAW: track 0.00 -> 109.0 mm
- net /VCO1_MOD: track 0.00 -> 85.8 mm
- net +15V: track 724.5 -> 802.5 mm
- net /S2: track 0.00 -> 74.3 mm
- net /R2: track 0.00 -> 66.5 mm
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