File: voicecard/voicecard.kicad_sch (KiCad schematic)
At the start: 187 parts, among them J2 Conn_01x25_Pin, J3 Conn_01x25_Pin, Q1 BF244C, Q2 BF244C, Q3 BF244C, Q4 BC212, Q5 BC212, Q6 BC212, Q7 BC212, Q8 BC212, Q9 BC212, U1 AS3340, U10 LM13700, U11 NE5532, U12 AS3310, U13 AS3310, U2 4016, U3 4016, U4 AS3340, U5 LM13700, U6 CA3080, U7 LM741, U8 LM13700, U9 NE5532

Commit message: Update voicecard layout
Parts:
- RV5: value 100k -> 22k
- renumbered R29 to R28, R28 to R29
Connections:
- net +15V: now also R91.2
- net -15V: no longer R91.2
- net -5V: now also CP16.2, CP29.2; no longer CP16.1, CP29.1
- net GND: now also CP16.1, CP29.1; no longer CP16.2, CP29.2
- net at R50.2, R53.1: now also U10.13 (-), U8.12
- net at R14.2, U11.6 (-): now also Q3.3 (S), R12.2, R13.1
- net at R10.2, U11.2 (-): now also Q2.3 (S), R11.1, R8.2
Other:
- moved on the sheet: CP16, CP29, R14
Changed lines of the file:
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@@
 	)
 	(junction
+		(at 420.37 160.02)
+		(diameter 0)
+		(color 0 0 0 0)
+	)
+	(junction
 		(at 341.63 330.2)
 		(diameter 0)
@@
 	)
 	(junction
+		(at 420.37 157.48)
+		(diameter 0)
+		(color 0 0 0 0)
+	)
+	(junction
 		(at 394.97 148.59)
 		(diameter 0)
@@
 	)
 	(junction
+		(at 478.79 163.83)
+		(diameter 0)
+		(color 0 0 0 0)
+	)
+	(junction
 		(at 416.56 137.16)
 		(diameter 0)
@@
 	)
 	(junction
+		(at 478.79 157.48)
+		(diameter 0)
+		(color 0 0 0 0)
+	)
+	(junction
 		(at 86.36 264.16)
 		(diameter 0)
@@
 	)
 	(junction
+		(at 372.11 135.89)
+		(diameter 0)
+		(color 0 0 0 0)
+	)
+	(junction
 		(at 86.36 67.31)
 		(diameter 0)
@@
 	(wire
 		(pts
-			(xy 379.73 135.89) (xy 365.76 135.89)
+			(xy 379.73 135.89) (xy 372.11 135.89)
 		)
 		(stroke
@@
 	(wire
 		(pts
-			(xy 372.11 124.46) (xy 372.11 151.13)
+			(xy 82.55 176.53) (xy 86.36 176.53)
 		)
 		(stroke
@@
 	(wire
 		(pts
-			(xy 82.55 176.53) (xy 86.36 176.53)
+			(xy 372.11 124.46) (xy 372.11 135.89)
 		)
 		(stroke
@@
 	(wire
 		(pts
-			(xy 480.06 163.83) (xy 482.6 163.83)
+			(xy 478.79 163.83) (xy 482.6 163.83)
 		)
 		(stroke
@@
 	(wire
 		(pts
+			(xy 372.11 135.89) (xy 365.76 135.89)
+		)
+		(stroke
+			(width 0)
+			(type default)
+		)
+	)
+	(wire
+		(pts
 			(xy 347.98 119.38) (xy 349.25 119.38)
 		)
@@
 	(wire
 		(pts
+			(xy 478.79 157.48) (xy 478.79 163.83)
+		)
+		(stroke
+			(width 0)
+			(type default)
+		)
+	)
+	(wire
+		(pts
 			(xy 382.27 184.15) (xy 382.27 185.42)
 		)
@@
 	(wire
 		(pts
+			(xy 372.11 135.89) (xy 372.11 151.13)
+		)
+		(stroke
+			(width 0)
+			(type default)
+		)
+	)
+	(wire
+		(pts
 			(xy 513.08 66.04) (xy 513.08 80.01)
 		)
@@
 	(wire
 		(pts
+			(xy 471.17 162.56) (xy 471.17 163.83)
+		)
+		(stroke
+			(width 0)
+			(type default)
+		)
+	)
+	(wire
+		(pts
 			(xy 461.01 372.11) (xy 461.01 369.57)
 		)
@@
 	(wire
 		(pts
+			(xy 420.37 157.48) (xy 420.37 160.02)
+		)
+		(stroke
+			(width 0)
+			(type default)
+		)
+	)
+	(wire
+		(pts
 			(xy 349.25 119.38) (xy 349.25 133.35)
 		)
@@
 	(wire
 		(pts
-			(xy 471.17 163.83) (xy 472.44 163.83)
+			(xy 467.36 162.56) (xy 471.17 162.56)
 		)
 		(stroke
@@
 	)
 	(label "KEY_PITCH"
-		(at 471.17 163.83 180)
+		(at 467.36 162.56 180)
 		(effects
 			(font
@@
 		)
 	)
-	(label "-15V"
+	(label "+15V"
 		(at 331.47 152.4 180)
 		(effects
@@
 	(symbol
 		(lib_id "Device:C_Polarized_Small")
-		(at 86.36 140.97 0)
+		(at 86.36 140.97 180)
 		(unit 1)
 		(exclude_from_sim no)
@@
 		(dnp no)
 		(property "Reference" "CP29"
-			(at 83.566 139.192 0)
+			(at 89.154 142.748 0)
 			(effects
 				(font
@@
 		)
 		(property "Value" "1uF"
-			(at 83.312 141.986 0)
+			(at 89.408 139.954 0)
 			(effects
 				(font
@@
 	(symbol
 		(lib_id "Device:C_Polarized_Small")
-		(at 86.36 274.32 0)
+		(at 86.36 274.32 180)
 		(unit 1)
 		(exclude_from_sim no)
@@
 		(dnp no)
 		(property "Reference" "CP16"
-			(at 83.566 272.542 0)
+			(at 89.154 276.098 0)
 			(effects
 				(font
@@
 		)
 		(property "Value" "1uF"
-			(at 83.312 275.336 0)
+			(at 89.408 273.304 0)
 			(effects
 				(font
@@
 		(dnp no)
 		(fields_autoplaced yes)
-		(property "Reference" "R28"
+		(property "Reference" "R29"
 			(at 538.48 91.4399 0)
 			(effects
@@
 			(project "voicecard"
 				(path "/13fddc44-f603-4567-a7d9-60d42f5208e5"
-					(reference "R28")
+					(reference "R29")
 					(unit 1)
 				)
@@
 		(fields_autoplaced yes)
 		(property "Reference" "RV5"
-			(at 107.95 64.7699 0)
+			(at 106.68 64.7699 0)
 			(effects
 				(font
@@
 			)
 		)
-		(property "Value" "100k"
-			(at 107.95 67.3099 0)
+		(property "Value" "22k"
+			(at 106.68 67.3099 0)
 			(effects
 				(font
@@
 		)
 		(property "Description" "HF TRACK"
-			(at 107.95 69.8499 0)
+			(at 106.68 69.8499 0)
 			(effects
 				(font
@@
 	(symbol
 		(lib_id "Device:R")
-		(at 476.25 163.83 90)
+		(at 474.98 163.83 90)
 		(unit 1)
 		(exclude_from_sim no)
@@
 		(fields_autoplaced yes)
 		(property "Reference" "R14"
-			(at 476.25 157.48 90)
+			(at 474.98 157.48 90)
 			(effects
 				(font
@@
 		)
 		(property "Value" "100k"
-			(at 476.25 160.02 90)
+			(at 474.98 160.02 90)
 			(effects
 				(font
@@
 		)
 		(property "Footprint" "Resistor_THT:R_Axial_DIN0309_L9.0mm_D3.2mm_P12.70mm_Horizontal"
-			(at 476.25 165.608 90)
+			(at 474.98 165.608 90)
 			(effects
 				(font
@@
 		)
 		(property "Datasheet" "~"
-			(at 476.25 163.83 0)
+			(at 474.98 163.83 0)
 			(effects
 				(font
@@
 		)
 		(property "Description" "Resistor"
-			(at 476.25 163.83 0)
+			(at 474.98 163.83 0)
 			(effects
 				(font
@@
 		(on_board yes)
 		(dnp no)
-		(property "Reference" "R29"
+		(property "Reference" "R28"
 			(at 458.47 132.0799 0)
 			(effects
@@
 			(project "voicecard"
 				(path "/13fddc44-f603-4567-a7d9-60d42f5208e5"
-					(reference "R29")
+					(reference "R28")
 					(unit 1)
 				)

Commit message: Update voicecard layout
Parts:
- CP14: footprint Capacitor_THT:CP_Radial_D5.0mm_P2.50mm -> Capacitor_THT:CP_Radial_D8.0mm_P3.50mm
- CP21: footprint Capacitor_THT:CP_Radial_D5.0mm_P2.50mm -> Capacitor_THT:CP_Radial_D8.0mm_P5.00mm
- CP22: footprint Capacitor_THT:CP_Radial_D5.0mm_P2.50mm -> Capacitor_THT:CP_Radial_D8.0mm_P3.80mm
- CP28: footprint Capacitor_THT:CP_Radial_D5.0mm_P2.50mm -> Capacitor_THT:CP_Radial_Tantal_D5.5mm_P5.00mm
- RV1, RV2, RV3, RV4, RV5, RV7, RV8: footprint Potentiometer_THT:Potentiometer_Bourns_3266Y_Vertical -> Potentiometer_THT:Potentiometer_Bourns_3299Y_Vertical
- RV6, RV9: footprint Potentiometer_THT:Potentiometer_Bourns_3266Y_Vertical -> Potentiometer_THT:Potentiometer_Bourns_3266P_Horizontal
Connections:
- net -15V: no longer U2.7 (VSS), U3.7 (VSS)
- net GND: now also U2.7 (VSS), U3.7 (VSS)
Other:
- note added: "On PCB R94 is after the junction, just before IC3 PIN 8"
Changed lines of the file:
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@@
 		)
 	)
+	(text "On PCB R94 is after \nthe junction, just \nbefore IC3 PIN 8"
+		(exclude_from_sim no)
+		(at 284.48 196.342 0)
+		(effects
+			(font
+				(size 1.27 1.27)
+			)
+		)
+	)
 	(junction
 		(at 307.34 88.9)
@@
 	(wire
 		(pts
-			(xy 269.24 187.96) (xy 269.24 190.5)
+			(xy 269.24 187.96) (xy 269.24 189.23)
 		)
 		(stroke
@@
 	)
 	(label "-15V"
-		(at 269.24 190.5 180)
+		(at 269.24 189.23 180)
 		(effects
 			(font
@@
 		)
 	)
-	(label "-15V"
-		(at 48.26 283.21 180)
+	(label "IC13_PIN14"
+		(at 365.76 311.15 0)
 		(effects
 			(font
 				(size 1.27 1.27)
 			)
-			(justify right bottom)
+			(justify left bottom)
 		)
 	)
-	(label "IC13_PIN14"
-		(at 365.76 311.15 0)
+	(label "GND"
+		(at 48.26 283.21 180)
 		(effects
 			(font
 				(size 1.27 1.27)
 			)
-			(justify left bottom)
+			(justify right bottom)
 		)
 	)
@@
 			)
 		)
-		(property "Footprint" "Potentiometer_THT:Potentiometer_Bourns_3266Y_Vertical"
+		(property "Footprint" "Potentiometer_THT:Potentiometer_Bourns_3266P_Horizontal"
 			(at 86.36 255.27 0)
 			(effects
@@
 			)
 		)
-		(property "Footprint" "Potentiometer_THT:Potentiometer_Bourns_3266Y_Vertical"
+		(property "Footprint" "Potentiometer_THT:Potentiometer_Bourns_3299Y_Vertical"
 			(at 104.14 196.85 0)
 			(effects
@@
 			)
 		)
-		(property "Footprint" "Potentiometer_THT:Potentiometer_Bourns_3266Y_Vertical"
+		(property "Footprint" "Potentiometer_THT:Potentiometer_Bourns_3299Y_Vertical"
 			(at 104.14 67.31 0)
 			(effects
@@
 			)
 		)
-		(property "Footprint" "Potentiometer_THT:Potentiometer_Bourns_3266Y_Vertical"
+		(property "Footprint" "Potentiometer_THT:Potentiometer_Bourns_3299Y_Vertical"
 			(at 528.32 66.04 0)
 			(effects
@@
 			)
 		)
-		(property "Footprint" "Capacitor_THT:CP_Radial_D5.0mm_P2.50mm"
+		(property "Footprint" "Capacitor_THT:CP_Radial_D8.0mm_P3.50mm"
 			(at 124.46 163.83 0)
 			(effects
@@
 			)
 		)
-		(property "Footprint" "Capacitor_THT:CP_Radial_D5.0mm_P2.50mm"
+		(property "Footprint" "Capacitor_THT:CP_Radial_D8.0mm_P5.00mm"
 			(at 317.5 153.67 0)
 			(effects
@@
 			)
 		)
-		(property "Footprint" "Potentiometer_THT:Potentiometer_Bourns_3266Y_Vertical"
+		(property "Footprint" "Potentiometer_THT:Potentiometer_Bourns_3299Y_Vertical"
 			(at 86.36 93.98 0)
 			(effects
@@
 			)
 		)
-		(property "Footprint" "Capacitor_THT:CP_Radial_D5.0mm_P2.50mm"
+		(property "Footprint" "Capacitor_THT:CP_Radial_D8.0mm_P3.80mm"
 			(at 312.42 116.84 0)
 			(effects
@@
 			)
 		)
-		(property "Footprint" "Capacitor_THT:CP_Radial_D5.0mm_P2.50mm"
+		(property "Footprint" "Capacitor_THT:CP_Radial_Tantal_D5.5mm_P5.00mm"
 			(at 123.19 25.4 0)
 			(effects
@@
 			)
 		)
-		(property "Footprint" "Potentiometer_THT:Potentiometer_Bourns_3266Y_Vertical"
+		(property "Footprint" "Potentiometer_THT:Potentiometer_Bourns_3299Y_Vertical"
 			(at 407.67 171.45 0)
 			(effects
@@
 			)
 		)
-		(property "Footprint" "Potentiometer_THT:Potentiometer_Bourns_3266Y_Vertical"
+		(property "Footprint" "Potentiometer_THT:Potentiometer_Bourns_3299Y_Vertical"
 			(at 393.7 78.74 0)
 			(effects
@@
 			)
 		)
-		(property "Footprint" "Potentiometer_THT:Potentiometer_Bourns_3266Y_Vertical"
+		(property "Footprint" "Potentiometer_THT:Potentiometer_Bourns_3266P_Horizontal"
 			(at 86.36 121.92 0)
 			(effects
@@
 			)
 		)
-		(property "Footprint" "Potentiometer_THT:Potentiometer_Bourns_3266Y_Vertical"
+		(property "Footprint" "Potentiometer_THT:Potentiometer_Bourns_3299Y_Vertical"
 			(at 86.36 223.52 0)
 			(effects
